File: hardware/keybit/keybit.kicad_pcb (KiCad board)
At the start: 2 copper layers, 19 x 19 mm, 15 parts, among them SW1 SW_Push, U1 CH32V003FxUx, U2 YZ13515055F-02025-02, U3 YZ13515055F-02025-02, U4 YZ13515055F-02025-02, U5 YZ13515055F-02025-02, U6 YZ13515055F-02025-02, U7 YZ13515055F-02025-02, U8 YZ13515055F-02025-02, U9 YZ13515055F-02025-02

Commit message: add in stuff
Parts:
- added R1: 4.7K, Resistor_SMD:R_0402_1005Metric, B.Cu at (145.0, 80.3)
- added R11: 4.7K, Resistor_SMD:R_0402_1005Metric, B.Cu at (153.1, 81.2)
- added R2: 4.7K, Resistor_SMD:R_0402_1005Metric, B.Cu at (145.0, 78.5)
- added R3: 4.7K, Resistor_SMD:R_0402_1005Metric, B.Cu at (147.0, 71.0)
- added R4: 4.7K, Resistor_SMD:R_0402_1005Metric, B.Cu at (154.9, 73.0)
- added R5: 4.7K, Resistor_SMD:R_0402_1005Metric, B.Cu at (150.9, 81.5)
- added R6: 4.7K, Resistor_SMD:R_0402_1005Metric, B.Cu at (145.2, 81.5)
- added R8: 4.7K, Resistor_SMD:R_0402_1005Metric, B.Cu at (153.1, 77.7)
Routing:
- net VCC: track 50.7 -> 61.7 mm, vias 4 -> 5
- net /SDA4: track 11.4 -> 14.7 mm
- net /SCL4: track 14.8 -> 16.4 mm
- net /SDA1: track 4.36 -> 5.91 mm
- net /SDA2: track 12.6 -> 13.4 mm
- net /SCL3: track 11.6 -> 12.5 mm
- net GND: track 11.3 -> 10.5 mm
- net /SCL2: track 7.59 -> 8.33 mm

Commit message: finished
Parts:
- moved R4 2.34 mm to (153.1, 74.5)
Connections:
- net VCC renamed +3.3V
Routing:
- net +3.3V: track 61.7 -> 63.0 mm
- net /SCL4: track 16.4 -> 16.9 mm
Other:
- outline, holes or cut-outs redrawn
- board text added: "Keybit"
