File: hardware/keybit/keybit.kicad_sch (KiCad schematic)
At the start: 15 parts, among them SW1 SW_Push, U1 CH32V003FxUx, U2 YZ13515055F-02025-02, U3 YZ13515055F-02025-02, U4 YZ13515055F-02025-02, U5 YZ13515055F-02025-02, U6 YZ13515055F-02025-02, U7 YZ13515055F-02025-02, U8 YZ13515055F-02025-02, U9 YZ13515055F-02025-02

Commit message: add in stuff
Parts:
- added R1, R11, R2, R3, R4, R5, R6, R8: 4.7K, Resistor_SMD:R_0402_1005Metric, symbol Device:R
Connections:
- net SCL1: now also R6.1
- net SCL2: now also R11.1
- net SCL3: now also R2.1
- net SCL4: now also R4.1
- net SDA1: now also R5.1
- net SDA2: now also R8.1
- net SDA3: now also R1.1
- net SDA4: now also R3.1
- net VCC: now also R1.2, R11.2, R2.2, R3.2, R4.2, R5.2, R6.2, R8.2

Commit message: finished
Connections:
- net VCC renamed +3.3V
Other:
- note added: "A modular keyboard key"
- note added: "CH32V003"
- note added: "Connectors"
- note added: "Keybit"
- note added: "Made by @notaroomba"
- moved on the sheet: C1, R1, R11, R2, R3, R4, R5, R6, R8, SW1, TP1, TP2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
