File: hardware/keybit/keybit.kicad_sch (KiCad schematic)
At the start: 23 parts, among them SW1 SW_Push, U1 CH32V003FxUx, U2 YZ13515055F-02025-02, U3 YZ13515055F-02025-02, U4 YZ13515055F-02025-02, U5 YZ13515055F-02025-02, U6 YZ13515055F-02025-02, U7 YZ13515055F-02025-02, U8 YZ13515055F-02025-02, U9 YZ13515055F-02025-02

Commit message: fixes adn stuff
Parts:
- R1, R11, R2, R3, R4, R5, R6, R8: value 4.7K -> 10K
Connections:
- net +3.3V: now also U7.1, U8.1; no longer U6.1, U9.1
- net GND: now also U6.2, U9.2; no longer U7.2, U8.2
- net SCL1: now also U9.1; no longer U8.1
- net SCL2: now also U6.1; no longer U7.1
- net SDA1: now also U8.2; no longer U9.2
- net SDA2: now also U7.2; no longer U6.2
- no-connect marks 6 -> 7
Other:
- moved on the sheet: U6, U7, U8, U9
