File: hardware/keyword/keyword.kicad_pcb (KiCad board)
At the start: 4 copper layers, 41.3 x 19 mm, 81 parts, among them CN1 YZ00615050R-08, CN2 YZ00615050R-08, CN3 YZ00615050R-08, CN4 YZ00615050R-08, CN5 YZ00615050R-08, CN6 YZ00615050R-08, CN7 YZ00615050R-08, CN8 YZ00615050R-08, CN9 YZ00615050R-08, U10 W25Q16JVUXIQ, U11 STM32WB55RGVx, U12 MLPF-WB-04D3, U13 YZ13515055F-02025-02, U14 XL-1608RGBC, U15 YZ13515055F-02025-02, U16 XRTC252012S2R2MBCA, U17 SZYY0402Y_C434450, U18 TPS631000DRLR, U19 YZ37215050R-02025-05, U2 TPD2EUSB30, U20 YZ37215050R-02025-05, U3 NX2012SA-32.768KHZ-STD-MUB-2, U4 YZ13515055F-02025-02, U5 YZ13515055F-02025-02, U6 YZ13515055F-02025-02, U7 YZ13515055F-02025-02, U8 BQ25895RTW, U9 DFE252012P-1R0M=P2, X1 NX2016SA-32MHZ-STD-CZS-5

Commit message: finished stuff
Parts:
- moved R1 0.25 mm to (185.6, 84.5)
- moved R2 0.19 mm to (189.8, 84.6)
- moved USB1 0.14 mm to (187.5, 88.1)
Other:
- outline, holes or cut-outs redrawn

Commit message: fixes adn stuff
Parts:
- removed C1, C2: 10pF, Capacitor_SMD:C_0402_1005Metric
- removed U17: SZYY0402Y_C434450, lcsc:LED0402-FD_YELLOW
- added C37: 10uF, Capacitor_SMD:C_0603_1608Metric, B.Cu at (190.4, 84.5)
- C6, C9: value 10pF -> 12pF
- R11, R8: value 4.7K -> 10K
- moved C16 0.62 mm to (187.7, 86.1)
Connections:
- U4 pad 1: +3.3V -> /SCL
- U4 pad 2: /SDA -> GND
- U7 pad 1: /SCL -> +3.3V
- U7 pad 2: GND -> /SDA
- U8 pad 23: unconnected-(U8-PMID-Pad23) -> Net-(U8-PMID)
- U8 pad 4: Net-(U17-K) -> unconnected-(U8-STAT-Pad4)
- U8 pad 5: /SDA -> /SCL
- U8 pad 6: /SCL -> /SDA
Routing:
- net Net-(U17-K): track 12.4 -> 0.00 mm, vias 2 -> 0
- net VCC: track 27.8 -> 16.3 mm
- net /SDA: track 61.6 -> 64.7 mm
- net /SCL: track 64.9 -> 67.7 mm
- net Net-(U8-PMID): track 0.00 -> 1.91 mm
- net /HXOUT: track 6.10 -> 4.28 mm
- net /HXIN: track 3.12 -> 1.90 mm
- net +3.3V: track 60.1 -> 59.0 mm
