File: hardware/keyword/keyword.kicad_sch (KiCad schematic)
At the start: 81 parts, among them CN1 YZ00615050R-08, CN2 YZ00615050R-08, CN3 YZ00615050R-08, CN4 YZ00615050R-08, CN5 YZ00615050R-08, CN6 YZ00615050R-08, CN7 YZ00615050R-08, CN8 YZ00615050R-08, CN9 YZ00615050R-08, U10 W25Q16JVUXIQ, U11 STM32WB55RGVx, U12 MLPF-WB-04D3, U13 YZ13515055F-02025-02, U14 XL-1608RGBC, U15 YZ13515055F-02025-02, U16 XRTC252012S2R2MBCA, U17 SZYY0402Y_C434450, U18 TPS631000DRLR, U19 YZ37215050R-02025-05, U2 TPD2EUSB30, U20 YZ37215050R-02025-05, U3 NX2012SA-32.768KHZ-STD-MUB-2, U4 YZ13515055F-02025-02, U5 YZ13515055F-02025-02, U6 YZ13515055F-02025-02, U7 YZ13515055F-02025-02, U8 BQ25895RTW, U9 DFE252012P-1R0M=P2, X1 NX2016SA-32MHZ-STD-CZS-5

Commit message: finished stuff
Parts:
- R12, R13, R14, R4, R5, R6, R7: LCSC C25082 -> (none)

Commit message: fixes adn stuff
Parts:
- removed U17: SZYY0402Y_C434450, lcsc:LED0402-FD_YELLOW, symbol lcsc:SZYY0402Y_C434450
- added C37: 10uF, Capacitor_SMD:C_0603_1608Metric, symbol Device:C
- C1, C2: now not fitted; now left out of the parts list
- C6, C9: value 10pF -> 12pF
- R11, R8: value 4.7K -> 10K
Connections:
- net +3.3V: now also U7.1; no longer U4.1
- net GND: now also U4.2, C37.2; no longer U7.2
- net SCL: now also U4.1, U8.5 (SCL); no longer U7.1, U8.6 (SDA)
- net SDA: now also U7.2, U8.6 (SDA); no longer U4.2, U8.5 (SCL)
- net at U8.23 (PMID): now also C37.1
Other:
- moved on the sheet: C16, C17, C18, C19, C20, C23, R4, R5, R6, R7, TP4, TP5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
